Commit message: Added vgdtas_tasks package

File: src/vgdtas_description/models/robot.urdf (robot description, URDF)
Before this commit: robot vgdtas_system, 38 links, 37 joints
Joints:
- joint fer_table_joint: origin xyz=-0.6 0 0 rpy=0 0 0 -> xyz=-0.7 0 0 rpy=0 0 0
- joint ur_table_joint: origin xyz=0.6 0 0 rpy=0 0 0 -> xyz=0.7 0 0 rpy=0 0 0

Commit message: Fixed urdf to spawn single-sided aruco marker and added filter to perception node

File: src/vgdtas_description/models/robot.urdf (robot description, URDF)
Before this commit: robot vgdtas_system, 38 links, 37 joints
Links:
- added link ur_aruco_cube_link; visual box size=0.05 0.05 0.049
- link ur_aruco_marker_link: geometry visual box size=0.05 0.05 0.001
Joints:
- added joint ur_aruco_cube_joint: type fixed, parent ur_tool0, child ur_aruco_cube_link, origin xyz=0.0 0.0 0.1595 rpy=0.0 0.0 0.0
- joint ur_aruco_marker_joint: origin xyz=0.0 0.0 0.16 rpy=0.0 0.0 0.0 -> xyz=0.0 0.0 0.025 rpy=0.0 0.0 0.0; parent ur_tool0 -> ur_aruco_cube_link

Commit message: Fixed frame issues in fer_perception_node

File: src/vgdtas_description/models/robot.urdf (robot description, URDF)
Before this commit: robot vgdtas_system, 39 links, 38 joints
Links:
- link ur_table: geometry collision box size=0.8 0.8 0.05; collision cylinder length=0.825 radius=0.03
Joints:
- joint ur_base_joint: origin xyz=0 0 0.75 rpy=0 0 0 -> xyz=0 0 0.85 rpy=0 0 0
